File: HARDWARE/V1/FC_H7_MINI/FC_H7_MINI.kicad_pcb (KiCad board)
At the start: 8 copper layers, 29 x 29 mm, 73 parts, among them IC1 ICM-42688-P, IC2 LMR51625YFDDCR, IC3 MX25R1635FZUIH0, IC4 LDL212PV33R, IC5 LDL212PV33R, J1 USB4110-GF-A, J2 SM08B-SRSS-TB, J3 SM06B-SRSS-TB, Q1 2N7002KQBZ, U2 STM32G473CEUx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

Commit message: up
Parts:
- added +5V1: TestPoint, samacsys2:PAD_1.5mmx1.5mm, B.Cu at (89.0, 99.4)
- added +5V2: TestPoint, samacsys2:PAD_1.5mmx1.5mm, B.Cu at (85.0, 101.4)
- added 5v1: TestPoint_Small, samacsys2:PAD_1.5mmx1.5mm_hole, F.Cu at (83.1, 105.5)
- added ADC_CURR1: TestPoint_Small, samacsys2:PAD_1.5mmx1.5mm_hole, F.Cu at (94.6, 74.5)
- added BUZ-1: TestPoint, samacsys2:PAD_1.5mmx1.5mm, B.Cu at (91.0, 99.4)
- added GND2: TestPoint, samacsys2:PAD_1.5mmx1.5mm, B.Cu at (87.0, 101.4)
- added GND9: TestPoint, samacsys2:PAD_1.5mmx1.5mm_hole, F.Cu at (92.3, 105.5)
- added LED1: TestPoint, samacsys2:1mm_circle, B.Cu at (103.8, 78.6)
- added LED2: TestPoint, samacsys2:1mm_circle, B.Cu at (101.5, 103.8)
- added LED3: TestPoint, samacsys2:1mm_circle, B.Cu at (76.3, 101.6)
- added LED4: TestPoint, samacsys2:1mm_circle, B.Cu at (78.3, 76.3)
- added LED5V1: TestPoint, samacsys2:1mm_circle, B.Cu at (76.3, 78.3)
- added LED5V2: TestPoint, samacsys2:1mm_circle, B.Cu at (101.7, 76.3)
- added LED5V3: TestPoint, samacsys2:1mm_circle, B.Cu at (103.8, 101.4)
- added LED5V4: TestPoint, samacsys2:1mm_circle, B.Cu at (78.4, 103.7)
- added LEDGND1: TestPoint, samacsys2:1mm_circle, B.Cu at (77.1, 77.1)
- added LEDGND2: TestPoint, samacsys2:1mm_circle, B.Cu at (103.0, 77.2)
- added LEDGND3: TestPoint, samacsys2:1mm_circle, B.Cu at (102.9, 102.9)
- added LEDGND4: TestPoint, samacsys2:1mm_circle, B.Cu at (77.1, 102.9)
- added M1: TestPoint_Small, samacsys2:PAD_1.5mmx1.5mm_hole, F.Cu at (85.4, 74.5)
- added M2: TestPoint_Small, samacsys2:PAD_1.5mmx1.5mm_hole, F.Cu at (87.7, 74.5)
- added M3: TestPoint_Small, samacsys2:PAD_1.5mmx1.5mm_hole, F.Cu at (90.0, 74.5)
- added M4: TestPoint_Small, samacsys2:PAD_1.5mmx1.5mm_hole, F.Cu at (92.3, 74.5)
- added RX4: TestPoint, samacsys2:PAD_1.5mmx1.5mm, B.Cu at (95.0, 101.4)
- added Rx2: TestPoint_Small, samacsys2:PAD_1.5mmx1.5mm_hole, F.Cu at (90.0, 105.5)
- added Rx3: TestPoint_Small, samacsys2:PAD_1.5mmx1.5mm_hole, F.Cu at (96.9, 74.5)
- added SCL1: TestPoint, samacsys2:PAD_1.5mmx1.5mm, B.Cu at (89.0, 101.4)
- added SDA1: TestPoint, samacsys2:PAD_1.5mmx1.5mm, B.Cu at (91.0, 101.4)
- added SWCLK1: TestPoint, samacsys2:1mm_circle, B.Cu at (87.7, 97.4)
- added SWDIO1: TestPoint, samacsys2:1mm_circle, B.Cu at (87.7, 96.0)
- added TX4: TestPoint, samacsys2:PAD_1.5mmx1.5mm, B.Cu at (93.0, 101.4)
- added Tx3: TestPoint_Small, samacsys2:PAD_1.5mmx1.5mm_hole, F.Cu at (99.2, 74.5)
- added USB5V1: TestPoint, samacsys2:PAD_1.5mmx1.5mm, B.Cu at (79.1, 86.3)
- added USBDM1: TestPoint, samacsys2:PAD_1.5mmx1.5mm, B.Cu at (79.1, 88.8)
- added USBDP1: TestPoint, samacsys2:PAD_1.5mmx1.5mm, B.Cu at (79.1, 91.3)
- added USBGND1: TestPoint, samacsys2:PAD_1.5mmx1.5mm, B.Cu at (79.1, 93.8)
- added VBAT+1: TestPoint_Small, samacsys2:PAD_1.5mmx1.5mm_hole, F.Cu at (83.1, 74.5)
- added gnd1: TestPoint_Small, samacsys2:PAD_1.5mmx1.5mm_hole, F.Cu at (80.8, 74.5)
- added gnd3: TestPoint_Small, samacsys2:PAD_1.5mmx1.5mm_hole, F.Cu at (85.4, 105.5)
- added rx1: TestPoint_Small, samacsys2:PAD_1.5mmx1.5mm_hole, F.Cu at (94.6, 105.5)
- added tx1: TestPoint_Small, samacsys2:PAD_1.5mmx1.5mm_hole, F.Cu at (96.9, 105.5)
- added tx2: TestPoint_Small, samacsys2:PAD_1.5mmx1.5mm_hole, F.Cu at (87.7, 105.5)
- IC4, IC5: footprint samacsys:SON50P200X200X80-7N-D -> samacsys2:SON50P200X200X80-7N-D
- moved R2 4.94 mm to (94.8, 81.8)
- moved C25 3.80 mm to (83.9, 90.3)
- moved C4 1.81 mm to (84.8, 82.6), turned to 180 degrees
- moved C12 1.15 mm to (90.5, 81.9)
- moved R5 1.13 mm to (86.5, 91.0)
- moved C13 0.95 mm to (84.8, 84.5)
- moved C5 0.91 mm to (85.7, 86.0)
- moved R1 0.80 mm to (83.9, 85.9)
- moved S3 0.66 mm to (94.8, 101.5)
- moved R11 0.66 mm to (88.8, 81.9)
- moved IC3 0.27 mm to (85.2, 88.7), turned to 180 degrees
- moved C17 0.25 mm to (97.5, 85.2)
- moved C8 0.25 mm to (99.5, 85.2)
- moved Y2 0.20 mm to (98.8, 93.9)
- moved C2 0.20 mm to (87.3, 95.5), turned to -90 degrees
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Connections:
- J3 pad 1: +12V -> +5V
- U2 pad 2: unconnected-(U2-PC13-Pad2) -> IMU_CLK_EXTI
- U2 pad 3: unconnected-(U2-PC14-Pad3) -> GYROEXTI
- U2 pad 4: unconnected-(U2-PC15-Pad4) -> GYRO_CS/SPI1
Routing:
- net VUSB: track 0.00 -> 16.0 mm, vias 0 -> 4
- net 4.5V: track 0.00 -> 10.6 mm
- net Rx1: track 0.00 -> 8.25 mm, vias 0 -> 1
- net Net-(IC2-FB): track 0.00 -> 7.90 mm
- net FLASH_MOSI/SPI2: track 0.00 -> 7.39 mm
- net Tx2: track 0.00 -> 6.30 mm
- net Rx2: track 0.00 -> 6.26 mm
- net FLASH_MISO/SPI2: track 0.00 -> 5.31 mm
- net Net-(J1-D+-PadA6): track 0.00 -> 5.14 mm, vias 0 -> 2
- net FLASH_CS/SPI2: track 0.00 -> 4.75 mm
- net Net-(J1-D--PadA7): track 0.00 -> 4.64 mm, vias 0 -> 2
- net HSE_IN: track 0.00 -> 4.39 mm
- net Net-(IC2-SW): track 0.00 -> 4.31 mm
- net Net-(J1-CC1): track 0.00 -> 4.30 mm
- net Net-(Q1-G): track 0.00 -> 4.02 mm
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Other:
- board size 29 x 29 mm -> 29 x 33 mm

Commit message: up
Parts:
- moved LEDBLUE1 1.55 mm to (83.7, 97.5)
- moved LEDGREEN1 1.55 mm to (85.2, 97.5)
- moved R5 1.23 mm to (87.5, 91.5)
- moved C6 0.60 mm to (96.9, 96.8), turned to 0 degrees
- moved Y2 0.27 mm to (98.8, 93.7)
- moved C11 0.20 mm to (98.0, 96.0)
- moved R13 0.10 mm to (87.5, 92.9)
- moved R6 0.10 mm to (87.5, 92.2)
- moved C2 0.10 mm to (87.3, 95.6)
- moved C9 0.10 mm to (87.5, 94.3)
- moved R22 0.10 mm to (88.2, 95.6)
- moved R61 0.10 mm to (87.5, 93.6)
Routing:
- net +5V: track 0.00 -> 39.8 mm, vias 8 -> 12
- net 3.3VMCU: track 0.00 -> 38.1 mm, vias 0 -> 7
- net Net-(J2-Pad6): track 0.00 -> 27.6 mm
- net Net-(J2-Pad5): track 0.00 -> 25.5 mm
- net Net-(J2-Pad4): track 0.00 -> 22.9 mm
- net 4.5V: track 10.6 -> 32.2 mm, vias 0 -> 4
- net Net-(J2-Pad3): track 0.00 -> 20.6 mm
- net Net-(LEDRED4-A): track 0.00 -> 18.9 mm
- net GYRO_MOSI/SPI1: track 1.40 -> 19.1 mm
- net I2C2_SDA: track 1.43 -> 14.9 mm
- net GYRO_MISO/SPI1: track 2.27 -> 15.1 mm
- net Tx1: track 0.67 -> 12.6 mm
- net IMU_CLK_EXTI: track 3.21 -> 15.2 mm
- net GYRO_SPI_CLK/SPI1: track 2.43 -> 14.1 mm
- net I2C2_SCL: track 2.08 -> 13.1 mm
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- added copper zone on F.Cu, net +5V
- added copper zone on F.Cu, net 3.3VMCU
- added copper zone on F.Cu, net 3.3VSENSOR
- added copper zone on B.Cu, net GND
- added copper zone on F.Cu, net GND
- added copper zone on In1.Cu, net GND
- added copper zone on In3.Cu, net GND
- added copper zone on F.Cu, net Net-(C17-Pad1)
- added copper zone on F.Cu, net Net-(IC2-SW)
- added copper zone on F.Cu, net VBAT+
Other:
- copper layers 8 -> 6

Commit message: up
Parts:
- removed LED2, LED3, LED4, LED5V1, LED5V2, LED5V3, LED5V4, LEDGND1, LEDGND2, LEDGND3, LEDGND4: TestPoint, samacsys2:1mm_circle
- added +5V2: TestPoint, samacsys2:PAD_1.5mmx1.5mm, B.Cu at (85.0, 99.4)
- added D1: SP3222-02ETG, samacsys2:SP322202ETG, F.Cu at (83.8, 90.7)
- added G***: LOGO, LOGO, B.Cu at (90.0, 86.0)
- added GND4: TestPoint, samacsys2:PAD_1.5mmx1.5mm, B.Cu at (87.0, 99.4)
- added PIO1: TestPoint, samacsys2:PAD_1.5mmx1.5mm, B.Cu at (95.0, 99.4)
- J1: footprint Connector_USB:USB_C_Receptacle_GCT_USB4110 -> Connector_USB:USB_C_Receptacle_GCT_USB4105-xx-A_16P_TopMnt_Horizontal
- LED1: footprint samacsys2:1mm_circle -> samacsys2:PAD_1.5mmx1.5mm
- moved LED1 25.5 mm to (89.0, 99.4), turned to -90 degrees
- moved C5 5.65 mm to (84.0, 80.6), turned to 90 degrees
- moved +5V1 4.00 mm to (93.0, 99.4)
- moved SWCLK1 3.11 mm to (88.0, 94.3)
- moved R10 1.60 mm to (85.5, 91.0)
- moved C27 0.79 mm to (94.3, 87.2), turned to 0 degrees
- moved C25 0.66 mm to (84.0, 89.7)
- moved IC3 0.60 mm to (85.2, 88.0)
- moved R14 0.60 mm to (93.1, 87.0)
- moved C10 0.60 mm to (89.9, 87.0)
- moved C16 0.60 mm to (91.7, 87.0)
- moved C24 0.60 mm to (91.0, 87.0)
- moved C26 0.60 mm to (92.4, 87.0)
- moved R8 0.45 mm to (94.3, 86.5), turned to 0 degrees
- moved SWDIO1 0.42 mm to (88.0, 95.7)
- renumbered +5V2 to +4.5V2, RX4 to RX2, Rx2 to Rx4, TX4 to TX2, tx2 to tx4
Connections:
- +4.5V2 pad 1: +5V -> 4.5V
- J3 pad 3: Tx2 -> Tx4
- J3 pad 4: Rx2 -> Rx4
- RX2 pad 1: Rx4 -> Rx2
- Rx4 pad 1: Rx2 -> Rx4
- TX2 pad 1: Tx4 -> Tx2
- U2 pad 12: unconnected-(U2-PA4-Pad12) -> PIO
- tx4 pad 1: Tx2 -> Tx4
Routing:
- net 3.3VMCU: track 38.1 -> 7.91 mm
- net Rx3: track 0.69 -> 26.4 mm
- net ESC_Curr: track 0.00 -> 19.7 mm
- net 4.5V: track 32.2 -> 12.5 mm, vias 4 -> 8
- net +5V: track 39.8 -> 20.5 mm, vias 12 -> 9
- net Tx3: track 0.72 -> 20.0 mm
- net Net-(J2-Pad3): track 20.6 -> 33.1 mm
- net PIO: track 0.00 -> 11.5 mm, vias 0 -> 2
- net Net-(J2-Pad6): track 27.6 -> 38.4 mm
- net Net-(J2-Pad4): track 22.9 -> 33.6 mm
- net Net-(J2-Pad5): track 25.5 -> 35.9 mm
- net GND: track 0.00 -> 10.3 mm, vias 136 -> 189
- net Tx4: track 9.28 -> 18.1 mm, vias 5 -> 1
- net Rx4: track 10.1 -> 17.3 mm, vias 5 -> 1
- net ADC_VBAT: track 3.00 -> 8.17 mm, vias 1 -> 2
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- added copper zone on In4.Cu, net +5V
- added copper zone on In4.Cu, net 3.3VMCU
- added copper zone on F.Cu, net 4.5V
- added copper zone on In4.Cu, net 4.5V
- added copper zone on B.Cu, net BUZ-
- added copper zone on B.Cu, net Net-(LED1-Pad1)
- added copper zone on In2.Cu, net Rx2
- added copper zone on In2.Cu, net Tx2
Other:
- board text added: "1"
- board text added: "2"
- board text added: "3"
- board text added: "4"
- board text added: "4.5V 5V"
- board text added: "5V"
- board text added: "Curr"
- board text added: "D+"
- board text added: "D-"
- board text added: "DJI"
- board text added: "Designed by : M.Pommery"
- board text added: "ESC"
- board text added: "Gnd"
- board text added: "Gnd Gnd"
- board text added: "M1"
- board text added: "M2"
- board text added: "M3"
- board text added: "M4"
- board text added: "Rx1"
- board text added: "Rx2 PIO"
- board text added: "Rx3"
- board text added: "Rx4"
- board text added: "Scl2 LED"
- board text added: "Sda2 Buz-"
- board text added: "Tx1"
- board text added: "Tx2 5V"
- board text added: "Tx3"
- board text added: "Tx4"
- board text added: "Vbat"
- board text added: "dio clk"
