File: HARDWARE/V1/FC_H7_MINI/FC_H7_MINI.kicad_sch (KiCad schematic)
At the start: 26 parts, among them Q1 2N7002KQBZ, U2 STM32G473CEUx, Y2 CSTNE8M00GH5C000R0

Commit message: up
Parts:
- Q1: footprint 2N7002KQBZ -> samacsys:2N7002KQBZ
Connections:
- net GYROEXTI: now also U2.3 (PC14)
- net GYRO_CS/SPI1: now also U2.4 (PC15)
- net IMU_CLK_EXTI: now also U2.2 (PC13)
- no-connect marks 0 -> 3
Changed lines of the file:
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@@
 		(color 0 0 0 0)
 	)
+	(no_connect
+		(at 209.55 120.65)
+	)
+	(no_connect
+		(at 209.55 100.33)
+	)
+	(no_connect
+		(at 245.11 92.71)
+	)
 	(wire
 		(pts
@@
 	(global_label "IMU_CLK_EXTI"
 		(shape input)
-		(at 153.67 114.3 180)
+		(at 209.55 110.49 180)
 		(fields_autoplaced yes)
 		(effects
@@
 		)
 		(property "Intersheetrefs" "${INTERSHEET_REFS}"
-			(at 137.8639 114.3 0)
+			(at 193.7439 110.49 0)
 			(effects
 				(font
@@
 	(global_label "GYRO_CS{slash}SPI1"
 		(shape input)
-		(at 153.67 121.92 180)
+		(at 209.55 115.57 180)
 		(fields_autoplaced yes)
 		(effects
@@
 		)
 		(property "Intersheetrefs" "${INTERSHEET_REFS}"
-			(at 136.6543 121.92 0)
+			(at 192.5343 115.57 0)
 			(effects
 				(font
@@
 	(global_label "GYROEXTI"
 		(shape input)
-		(at 153.67 111.76 180)
+		(at 209.55 113.03 180)
 		(fields_autoplaced yes)
 		(effects
@@
 		)
 		(property "Intersheetrefs" "${INTERSHEET_REFS}"
-			(at 141.7948 111.76 0)
+			(at 197.6748 113.03 0)
 			(effects
 				(font
@@
 			)
 		)
-		(property "Footprint" "2N7002KQBZ"
+		(property "Footprint" "samacsys:2N7002KQBZ"
 			(at 73.66 260.02 0)
 			(effects

Commit message: up
Connections:
- net PIO: now reaches U2.12 (PA4)
Other:
- moved on the sheet: C10, C11, C14, C16, C18, C19, C24, C26, C27, C6, C7, C9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
