File: HARDWARE/V1/FC_H7_MINI/untitled.kicad_sch (KiCad schematic)
At the start: 28 parts, among them IC2 LMR51625YFDDCR, IC4 LDL212PV33R, IC5 LDL212PV33R, J1 USB4110-GF-A

Commit message: up
Parts:
- added USB5V1, USBDM1, USBDP1, USBGND1: TestPoint, samacsys2:PAD_1.5mmx1.5mm, symbol Connector:TestPoint
- FB1: footprint BEADC2012X90N -> samacsys2:BEADC2012X90N
- IC4, IC5: footprint SON50P200X200X80-7N-D -> samacsys2:SON50P200X200X80-7N-D
Connections:
- net GND: now also USBGND1.1
- net VUSB: now also USB5V1.1
- net at J1.A6 (D+), J1.B6 (D+), R61.1: now also USBDP1.1
- net at J1.A7 (D-), J1.B7 (D-), R13.1: now also USBDM1.1

Commit message: up
Parts:
- added D1: SP3222-02ETG, samacsys2:SP322202ETG, symbol samacsys2:SP3222-02ETG
- J1: footprint Connector_USB:USB_C_Receptacle_GCT_USB4110 -> Connector_USB:USB_C_Receptacle_GCT_USB4105-xx-A_16P_TopMnt_Horizontal
Connections:
- net GND: now also D1.3 (GND)
- net at J1.A6 (D+), J1.B6 (D+), R61.1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: now also D1.2 (K_2)
- net at J1.A7 (D-), J1.B7 (D-), R13.1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: now also D1.1 (K_1)
Other:
- note added: "SP3222-02ETG"
- moved on the sheet: C1, C12, C13, C17, C2, C23, C3, C4, C5, C8, D10, D11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
