File: HARDWARE/V1/MINIREX_G4/Peripherials.kicad_sch (KiCad schematic)
At the start: 8 parts, among them IC1 ICM-42688-P, IC3 MX25R1635FZUIH0

Commit message: up
Parts:
- C20, C21, C22, C25: symbol Device:C_Small -> minirex_g4:C_Small
- IC1: symbol Samacsys_Parts:ICM-42688-P -> minirex_g4:ICM-42688-P
- IC3: symbol samacsys2:MX25R1635FZUIH0 -> minirex_g4:MX25R1635FZUIH0
- R15: symbol Device:R_Small -> minirex_g4:R_Small_1
- R9: symbol Device:R_Small -> minirex_g4:R_Small
Changed lines of the file:
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@@
 	)
 	(symbol
-		(lib_id "Device:C_Small")
+		(lib_id "minirex_g4:C_Small")
 		(at 171.45 134.62 0)
 		(unit 1)
@@
 	)
 	(symbol
-		(lib_id "power:GND")
+		(lib_id "minirex_g4:GND")
 		(at 80.01 106.68 0)
 		(unit 1)
@@
 	)
 	(symbol
-		(lib_id "Device:R_Small")
+		(lib_id "minirex_g4:R_Small")
 		(at 209.55 121.92 180)
 		(unit 1)
@@
 	)
 	(symbol
-		(lib_id "power:GND")
+		(lib_id "minirex_g4:GND")
 		(at 171.45 137.16 0)
 		(unit 1)
@@
 	(symbol
 		(lib_name "R_Small_1")
-		(lib_id "Device:R_Small")
+		(lib_id "minirex_g4:R_Small_1")
 		(at 86.36 35.56 90)
 		(unit 1)
@@
 	)
 	(symbol
-		(lib_id "power:GND")
+		(lib_id "minirex_g4:GND")
 		(at 77.47 106.68 0)
 		(unit 1)
@@
 	)
 	(symbol
-		(lib_id "power:GND")
+		(lib_id "minirex_g4:GND")
 		(at 125.73 95.25 0)
 		(unit 1)
@@
 	)
 	(symbol
-		(lib_id "Device:C_Small")
+		(lib_id "minirex_g4:C_Small")
 		(at 130.81 92.71 0)
 		(unit 1)
@@
 	)
 	(symbol
-		(lib_id "Samacsys_Parts:ICM-42688-P")
+		(lib_id "minirex_g4:ICM-42688-P")
 		(at 44.45 81.28 0)
 		(unit 1)
@@
 	)
 	(symbol
-		(lib_id "power:GND")
+		(lib_id "minirex_g4:GND")
 		(at 209.55 135.89 270)
 		(unit 1)
@@
 	)
 	(symbol
-		(lib_id "Device:C_Small")
+		(lib_id "minirex_g4:C_Small")
 		(at 67.31 114.3 0)
 		(unit 1)
@@
 	)
 	(symbol
-		(lib_id "power:GND")
+		(lib_id "minirex_g4:GND")
 		(at 232.41 148.59 0)
 		(unit 1)
@@
 	)
 	(symbol
-		(lib_id "power:GND")
+		(lib_id "minirex_g4:GND")
 		(at 110.49 81.28 90)
 		(unit 1)
@@
 	)
 	(symbol
-		(lib_id "samacsys2:MX25R1635FZUIH0")
+		(lib_id "minirex_g4:MX25R1635FZUIH0")
 		(at 209.55 128.27 0)
 		(unit 1)
@@
 	)
 	(symbol
-		(lib_id "power:GND")
+		(lib_id "minirex_g4:GND")
 		(at 67.31 116.84 0)
 		(unit 1)
@@
 	)
 	(symbol
-		(lib_id "Device:C_Small")
+		(lib_id "minirex_g4:C_Small")
 		(at 116.84 92.71 0)
 		(unit 1)

Commit message: up
Parts:
- IC3: Mouser Part Number (none) -> 95-25R1635FZUIH0TR
Changed lines of the file:
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@@
+			)
+		)
+		(property "Field5" ""
+			(at 171.45 134.62 0)
+			(effects
+				(font
+					(size 1.27 1.27)
+				)
+				(hide yes)
+			)
+		)
+		(property "PRICE(1U)" ""
+			(at 171.45 134.62 0)
+			(effects
+				(font
+					(size 1.27 1.27)
+				)
+				(hide yes)
+			)
+		)
+		(property "PRICE(100u)" ""
+			(at 171.45 134.62 0)
+			(effects
+				(font
+					(size 1.27 1.27)
+				)
+				(hide yes)
 			)
 		)
@@
 		)
 		(property "Manufacturer_Name" "Panasonic"
+			(at 209.55 121.92 0)
+			(effects
+				(font
+					(size 1.27 1.27)
+				)
+				(hide yes)
+			)
+		)
+		(property "Field5" ""
+			(at 209.55 121.92 0)
+			(effects
+				(font
+					(size 1.27 1.27)
+				)
+				(hide yes)
+			)
+		)
+		(property "PRICE(1U)" ""
+			(at 209.55 121.92 0)
+			(effects
+				(font
+					(size 1.27 1.27)
+				)
+				(hide yes)
+			)
+		)
+		(property "PRICE(100u)" ""
 			(at 209.55 121.92 0)
 			(effects
@@
 			)
 		)
+		(property "Field5" ""
+			(at 86.36 35.56 0)
+			(effects
+				(font
+					(size 1.27 1.27)
+				)
+				(hide yes)
+			)
+		)
+		(property "PRICE(1U)" ""
+			(at 86.36 35.56 0)
+			(effects
+				(font
+					(size 1.27 1.27)
+				)
+				(hide yes)
+			)
+		)
+		(property "PRICE(100u)" ""
+			(at 86.36 35.56 0)
+			(effects
+				(font
+					(size 1.27 1.27)
+				)
+				(hide yes)
+			)
+		)
 		(pin "2"
 		)
@@
 			)
 		)
+		(property "Field5" ""
+			(at 130.81 92.71 0)
+			(effects
+				(font
+					(size 1.27 1.27)
+				)
+				(hide yes)
+			)
+		)
+		(property "PRICE(1U)" ""
+			(at 130.81 92.71 0)
+			(effects
+				(font
+					(size 1.27 1.27)
+				)
+				(hide yes)
+			)
+		)
+		(property "PRICE(100u)" ""
+			(at 130.81 92.71 0)
+			(effects
+				(font
+					(size 1.27 1.27)
+				)
+				(hide yes)
+			)
+		)
 		(pin "2"
 		)
@@
 			)
 		)
+		(property "Field5" ""
+			(at 44.45 81.28 0)
+			(effects
+				(font
+					(size 1.27 1.27)
+				)
+				(hide yes)
+			)
+		)
+		(property "PRICE(1U)" ""
+			(at 44.45 81.28 0)
+			(effects
+				(font
+					(size 1.27 1.27)
+				)
+				(hide yes)
+			)
+		)
+		(property "PRICE(100u)" ""
+			(at 44.45 81.28 0)
+			(effects
+				(font
+					(size 1.27 1.27)
+				)
+				(hide yes)
+			)
+		)
 		(pin "5"
 		)
@@
 			)
 		)
+		(property "Field5" ""
+			(at 67.31 114.3 0)
+			(effects
+				(font
+					(size 1.27 1.27)
+				)
+				(hide yes)
+			)
+		)
+		(property "PRICE(1U)" ""
+			(at 67.31 114.3 0)
+			(effects
+				(font
+					(size 1.27 1.27)
+				)
+				(hide yes)
+			)
+		)
+		(property "PRICE(100u)" ""
+			(at 67.31 114.3 0)
+			(effects
+				(font
+					(size 1.27 1.27)
+				)
+				(hide yes)
+			)
+		)
 		(pin "2"
 		)
@@
 			)
 		)
-		(property "Mouser Part Number" ""
+		(property "Mouser Part Number" "95-25R1635FZUIH0TR"
 			(at 251.46 823.19 0)
 			(effects
@@
 				)
 				(justify left top)
+				(hide yes)
+			)
+		)
+		(property "Field5" ""
+			(at 209.55 128.27 0)
+			(effects
+				(font
+					(size 1.27 1.27)
+				)
+				(hide yes)
+			)
+		)
+		(property "PRICE(1U)" ""
+			(at 209.55 128.27 0)
+			(effects
+				(font
+					(size 1.27 1.27)
+				)
+				(hide yes)
+			)
+		)
+		(property "PRICE(100u)" ""
+			(at 209.55 128.27 0)
+			(effects
+				(font
+					(size 1.27 1.27)
+				)
 				(hide yes)
 			)
@@
 			(at 116.84 92.71 0)
 			(effects
+				(font
+					(size 1.27 1.27)
+				)
+				(hide yes)
+			)
+		)
+		(property "Field5" ""
+			(at 116.84 92.71 0)
+			(effects
+				(font
+					(size 1.27 1.27)
+				)
+				(hide yes)
+			)
+		)
+		(property "PRICE(1U)" ""
+			(at 116.84 92.71 0)
+			(effects
+				(font
+					(size 1.27 1.27)
+				)
+				(hide yes)
+			)
+		)
+		(property "PRICE(100u)" ""
+			(at 116.84 92.71 0)
+			(effects
