File: HARDWARE/V1/MINIREX_G4/connectors.kicad_sch (KiCad schematic)
At the start: 41 parts, among them J2 SM08B-SRSS-TB, J3 SM06B-SRSS-TB, M1 TestPoint_Small, M2 TestPoint_Small, M3 TestPoint_Small, M4 TestPoint_Small

Commit message: up
Parts:
- +4.5V2, +5V1, +5V2, BUZ-1, GND2, GND4, GND9, LED1, Mounting_hole1, Mounting_hole2, Mounting_hole3, Mounting_hole4, PIO1, RX2, SCL1, SDA1, SWCLK1, SWDIO1, TX2: symbol Connector:TestPoint -> minirex_g4:TestPoint
- 5v1, ADC_CURR1, M1, M2, M3, M4, Rx3, Rx4, Tx3, VBAT+1, gnd1, gnd3, rx1, tx1, tx4: symbol Connector:TestPoint_Small -> minirex_g4:TestPoint_Small
- J2: symbol samacsys:SM08B-SRSS-TB -> minirex_g4:SM08B-SRSS-TB
- J3: symbol samacsys2:SM06B-SRSS-TB -> minirex_g4:SM06B-SRSS-TB
- R44: symbol Device:R_Small -> minirex_g4:R_Small_1
- R45: symbol Device:R_Small -> minirex_g4:R_Small_2
- R46: symbol Device:R_Small -> minirex_g4:R_Small_3
- R47: symbol Device:R_Small -> minirex_g4:R_Small_4
- R56: symbol Device:R_Small -> minirex_g4:R_Small
Changed lines of the file:
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@@
 	)
 	(symbol
-		(lib_id "Connector:TestPoint_Small")
+		(lib_id "minirex_g4:TestPoint_Small")
 		(at 57.15 33.02 0)
 		(unit 1)
@@
 	)
 	(symbol
-		(lib_id "Connector:TestPoint")
+		(lib_id "minirex_g4:TestPoint")
 		(at 91.44 73.66 0)
 		(unit 1)
@@
 	)
 	(symbol
-		(lib_id "Connector:TestPoint_Small")
+		(lib_id "minirex_g4:TestPoint_Small")
 		(at 54.61 35.56 0)
 		(unit 1)
@@
 	)
 	(symbol
-		(lib_id "Connector:TestPoint_Small")
+		(lib_id "minirex_g4:TestPoint_Small")
 		(at 146.05 33.02 0)
 		(unit 1)
@@
 	)
 	(symbol
-		(lib_id "Connector:TestPoint_Small")
+		(lib_id "minirex_g4:TestPoint_Small")
 		(at 49.53 25.4 0)
 		(mirror y)
@@
 	)
 	(symbol
-		(lib_id "Connector:TestPoint")
+		(lib_id "minirex_g4:TestPoint")
 		(at 78.74 100.33 0)
 		(unit 1)
@@
 	)
 	(symbol
-		(lib_id "power:GND")
+		(lib_id "minirex_g4:GND")
 		(at 114.3 74.93 0)
 		(unit 1)
@@
 	)
 	(symbol
-		(lib_id "Connector:TestPoint")
+		(lib_id "minirex_g4:TestPoint")
 		(at 29.21 100.33 0)
 		(unit 1)
@@
 	)
 	(symbol
-		(lib_id "power:GND")
+		(lib_id "minirex_g4:GND")
 		(at 86.36 34.29 0)
 		(unit 1)
@@
 	)
 	(symbol
-		(lib_id "power:GND")
+		(lib_id "minirex_g4:GND")
 		(at 53.34 48.26 270)
 		(unit 1)
@@
 	)
 	(symbol
-		(lib_id "Connector:TestPoint")
+		(lib_id "minirex_g4:TestPoint")
 		(at 132.08 100.33 0)
 		(unit 1)
@@
 	)
 	(symbol
-		(lib_id "Connector:TestPoint")
+		(lib_id "minirex_g4:TestPoint")
 		(at 72.39 73.66 0)
 		(unit 1)
@@
 	)
 	(symbol
-		(lib_id "power:GND")
+		(lib_id "minirex_g4:GND")
 		(at 135.89 74.93 0)
 		(unit 1)
@@
 	)
 	(symbol
-		(lib_id "Connector:TestPoint")
+		(lib_id "minirex_g4:TestPoint")
 		(at 176.53 100.33 0)
 		(unit 1)
@@
 	)
 	(symbol
-		(lib_id "Connector:TestPoint_Small")
+		(lib_id "minirex_g4:TestPoint_Small")
 		(at 53.34 30.48 0)
 		(unit 1)
@@
 	)
 	(symbol
-		(lib_id "power:+5V")
+		(lib_id "minirex_g4:+5V")
 		(at 144.78 33.02 90)
 		(unit 1)
@@
 	)
 	(symbol
-		(lib_id "Connector:TestPoint_Small")
+		(lib_id "minirex_g4:TestPoint_Small")
 		(at 146.05 35.56 0)
 		(unit 1)
@@
 	)
 	(symbol
-		(lib_id "power:GND")
+		(lib_id "minirex_g4:GND")
 		(at 144.78 35.56 270)
 		(unit 1)
@@
 	)
 	(symbol
-		(lib_id "power:GND")
+		(lib_id "minirex_g4:GND")
 		(at 175.26 38.1 0)
 		(unit 1)
@@
 	)
 	(symbol
-		(lib_id "Connector:TestPoint_Small")
+		(lib_id "minirex_g4:TestPoint_Small")
 		(at 146.05 38.1 0)
 		(unit 1)
@@
 	(symbol
 		(lib_name "R_Small_3")
-		(lib_id "Device:R_Small")
+		(lib_id "minirex_g4:R_Small_3")
 		(at 38.1 41.91 270)
 		(mirror x)
@@
 	(symbol
 		(lib_name "R_Small_1")
-		(lib_id "Device:R_Small")
+		(lib_id "minirex_g4:R_Small_1")
 		(at 38.1 30.48 270)
 		(mirror x)
@@
 	)
 	(symbol
-		(lib_id "Connector:TestPoint")
+		(lib_id "minirex_g4:TestPoint")
 		(at 152.4 100.33 0)
 		(unit 1)
@@
 	)
 	(symbol
-		(lib_id "power:+5V")
+		(lib_id "minirex_g4:+5V")
 		(at 176.53 100.33 180)
 		(unit 1)
@@
 	)
 	(symbol
-		(lib_id "power:GND")
+		(lib_id "minirex_g4:GND")
 		(at 127 43.18 270)
 		(unit 1)
@@
 	)
 	(symbol
-		(lib_id "Connector:TestPoint_Small")
+		(lib_id "minirex_g4:TestPoint_Small")
 		(at 54.61 45.72 0)
 		(unit 1)
@@
 	)
 	(symbol
-		(lib_id "Device:R_Small")
+		(lib_id "minirex_g4:R_Small")
 		(at 152.4 102.87 0)
 		(mirror y)
@@
 	)
 	(symbol
-		(lib_id "Connector:TestPoint")
+		(lib_id "minirex_g4:TestPoint")
 		(at 52.07 100.33 0)
 		(unit 1)
@@
 	)
 	(symbol
-		(lib_id "Connector:TestPoint")
+		(lib_id "minirex_g4:TestPoint")
 		(at 134.62 43.18 180)
 		(unit 1)
@@
 	)
 	(symbol
-		(lib_id "Connector:TestPoint")
+		(lib_id "minirex_g4:TestPoint")
 		(at 63.5 100.33 0)
 		(unit 1)
@@
 	)
 	(symbol
-		(lib_id "Connector:TestPoint_Small")
+		(lib_id "minirex_g4:TestPoint_Small")
 		(at 146.05 45.72 0)
 		(unit 1)
@@
 	)
 	(symbol
-		(lib_id "Connector:TestPoint")
+		(lib_id "minirex_g4:TestPoint")
 		(at 40.64 100.33 0)
 		(unit 1)
@@
 	)
 	(symbol
-		(lib_id "samacsys:SM08B-SRSS-TB")
+		(lib_id "minirex_g4:SM08B-SRSS-TB")
 		(at 86.36 30.48 0)
 		(mirror y)
@@
 	(symbol
 		(lib_name "R_Small_2")
-		(lib_id "Device:R_Small")
+		(lib_id "minirex_g4:R_Small_2")
 		(at 38.1 36.83 270)
 		(mirror x)
@@
 	)
 	(symbol
-		(lib_id "Connector:TestPoint_Small")
+		(lib_id "minirex_g4:TestPoint_Small")
 		(at 143.51 52.07 0)
 		(unit 1)
@@
 	)
 	(symbol
-		(lib_id "power:GND")
+		(lib_id "minirex_g4:GND")
 		(at 165.1 100.33 0)
 		(unit 1)
@@
 	)
 	(symbol
-		(lib_id "Connector:TestPoint")
+		(lib_id "minirex_g4:TestPoint")
 		(at 135.89 74.93 0)
 		(unit 1)
@@
 	)
 	(symbol
-		(lib_id "power:GND")
+		(lib_id "minirex_g4:GND")
 		(at 78.74 100.33 0)
 		(unit 1)
@@
 	)
 	(symbol
-		(lib_id "Connector:TestPoint")
+		(lib_id "minirex_g4:TestPoint")
 		(at 92.71 100.33 0)
 		(unit 1)
@@
 	)
 	(symbol
-		(lib_id "Connector:TestPoint_Small")
+		(lib_id "minirex_g4:TestPoint_Small")
 		(at 54.61 38.1 0)
 		(unit 1)
@@
 	)
 	(symbol
-		(lib_id "power:+5V")
+		(lib_id "minirex_g4:+5V")
 		(at 105.41 100.33 180)
 		(unit 1)
@@
 	)
 	(symbol
-		(lib_id "power:GND")
+		(lib_id "minirex_g4:GND")
 		(at 91.44 73.66 0)
 		(unit 1)
@@
 	(symbol
 		(lib_name "R_Small_4")
-		(lib_id "Device:R_Small")
+		(lib_id "minirex_g4:R_Small_4")
 		(at 38.1 46.99 270)
 		(mirror x)
@@
 	)
 	(symbol
-		(lib_id "Connector:TestPoint")
+		(lib_id "minirex_g4:TestPoint")
 		(at 165.1 100.33 0)
 		(unit 1)
@@
 	)
 	(symbol
-		(lib_id "Connector:TestPoint")
+		(lib_id "minirex_g4:TestPoint")
 		(at 114.3 74.93 0)
 		(unit 1)
@@
 	)
 	(symbol
-		(lib_id "Connector:TestPoint")
+		(lib_id "minirex_g4:TestPoint")
 		(at 118.11 100.33 0)
 		(unit 1)
@@
 	)
 	(symbol
-		(lib_id "Connector:TestPoint")
+		(lib_id "minirex_g4:TestPoint")
 		(at 105.41 100.33 0)
 		(unit 1)
@@
 	)
 	(symbol
-		(lib_id "Connector:TestPoint_Small")
+		(lib_id "minirex_g4:TestPoint_Small")
 		(at 146.05 40.64 0)
 		(unit 1)
@@
 	)
 	(symbol
-		(lib_id "Connector:TestPoint")
+		(lib_id "minirex_g4:TestPoint")
 		(at 189.23 100.33 0)
 		(unit 1)
@@
 	)
 	(symbol
-		(lib_id "Connector:TestPoint")
+		(lib_id "minirex_g4:TestPoint")
 		(at 17.78 100.33 0)
 		(unit 1)
@@
 	)
 	(symbol
-		(lib_id "power:GND")
+		(lib_id "minirex_g4:GND")
 		(at 72.39 73.66 0)
 		(unit 1)
@@
 	)
 	(symbol
-		(lib_id "Connector:TestPoint_Small")
+		(lib_id "minirex_g4:TestPoint_Small")
 		(at 53.34 43.18 0)
 		(unit 1)
@@
 	)
 	(symbol
-		(lib_id "Connector:TestPoint_Small")
+		(lib_id "minirex_g4:TestPoint_Small")
 		(at 54.61 40.64 0)
 		(unit 1)
@@
 	)
 	(symbol
-		(lib_id "Connector:TestPoint_Small")
+		(lib_id "minirex_g4:TestPoint_Small")
 		(at 54.61 48.26 0)
 		(unit 1)
@@
 	)
 	(symbol
-		(lib_id "samacsys2:SM06B-SRSS-TB")
+		(lib_id "minirex_g4:SM06B-SRSS-TB")
 		(at 175.26 33.02 0)
 		(mirror y)

Commit message: up
Parts:
- J2: Mouser Part Number N/A -> 306-SM08BSRSSTB
- J3: Mouser Part Number (none) -> 306-M06BSRSSTBLFSNPP
