File: HARDWARE/V1/MINIREX_G4/untitled.kicad_sch (KiCad schematic)
At the start: 33 parts, among them IC2 LMR51625YFDDCR, IC4 LDL212PV33R, IC5 LDL212PV33R, J1 USB4110-GF-A

Commit message: up
Parts:
- C1, C12, C13, C17, C2, C23, C3, C4, C5, C8: symbol Device:C_Small -> minirex_g4:C_Small
- D1: symbol samacsys2:SP3222-02ETG -> minirex_g4:SP3222-02ETG
- D10, D11: symbol samacsys:BAT60JFILM -> minirex_g4:BAT60JFILM
- FB1: symbol samacsys2:74279220800 -> minirex_g4:74279220800
- IC2: symbol samacsys:LMR51625YFDDCR -> minirex_g4:LMR51625YFDDCR
- IC4, IC5: symbol samacsys2:LDL212PV33R -> minirex_g4:LDL212PV33R
- J1: symbol Vraielogousbcwurth:USB_C_Receptacle_USB2.0_14P -> minirex_g4:USB_C_Receptacle_USB2.0_14P
- L1: symbol samacsys2:74479335329247 -> minirex_g4:74479335329247
- LEDRED3, LEDRED4: symbol Device:LED_Small -> minirex_g4:LED_Small
- R1: symbol Device:R_Small -> minirex_g4:R_Small_1
- R10: symbol Device:R_Small -> minirex_g4:R_Small_2
- R11: symbol Device:R_Small -> minirex_g4:R_Small_6
- R13: symbol Device:R_Small -> minirex_g4:R_Small_3
- R2: symbol Device:R_Small -> minirex_g4:R_Small_5
- R21: symbol Device:R_Small -> minirex_g4:R_Small_7
- R22: symbol Device:R_Small -> minirex_g4:R_Small
- R61: symbol Device:R_Small -> minirex_g4:R_Small_4
- USB5V1, USBDM1, USBDP1, USBGND1: symbol Connector:TestPoint -> minirex_g4:TestPoint
Changed lines of the file:
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@@
 	)
 	(symbol
-		(lib_id "power:GND")
+		(lib_id "minirex_g4:GND")
 		(at 68.58 135.89 0)
 		(unit 1)
@@
 	)
 	(symbol
-		(lib_id "Device:C_Small")
+		(lib_id "minirex_g4:C_Small")
 		(at 153.67 39.37 0)
 		(unit 1)
@@
 	)
 	(symbol
-		(lib_id "power:GND")
+		(lib_id "minirex_g4:GND")
 		(at 248.92 93.98 0)
 		(unit 1)
@@
 	)
 	(symbol
-		(lib_id "power:GND")
+		(lib_id "minirex_g4:GND")
 		(at 250.19 135.89 0)
 		(unit 1)
@@
 	)
 	(symbol
-		(lib_id "power:GND")
+		(lib_id "minirex_g4:GND")
 		(at 162.56 132.08 0)
 		(unit 1)
@@
 	)
 	(symbol
-		(lib_id "samacsys:BAT60JFILM")
+		(lib_id "minirex_g4:BAT60JFILM")
 		(at 248.92 45.72 180)
 		(unit 1)
@@
 	)
 	(symbol
-		(lib_id "Device:C_Small")
+		(lib_id "minirex_g4:C_Small")
 		(at 166.37 92.71 0)
 		(unit 1)
@@
 	)
 	(symbol
-		(lib_id "Device:C_Small")
+		(lib_id "minirex_g4:C_Small")
 		(at 162.56 129.54 0)
 		(unit 1)
@@
 	)
 	(symbol
-		(lib_id "samacsys2:LDL212PV33R")
+		(lib_id "minirex_g4:LDL212PV33R")
 		(at 210.82 124.46 0)
 		(mirror y)
@@
 	)
 	(symbol
-		(lib_id "Connector:TestPoint")
+		(lib_id "minirex_g4:TestPoint")
 		(at 93.98 85.09 0)
 		(unit 1)
@@
 	)
 	(symbol
-		(lib_id "Device:C_Small")
+		(lib_id "minirex_g4:C_Small")
 		(at 55.88 26.67 0)
 		(unit 1)
@@
 	(symbol
 		(lib_name "R_Small_6")
-		(lib_id "Device:R_Small")
+		(lib_id "minirex_g4:R_Small_6")
 		(at 137.16 50.8 0)
 		(unit 1)
@@
 	)
 	(symbol
-		(lib_id "power:GND")
+		(lib_id "minirex_g4:GND")
 		(at 242.57 116.84 90)
 		(unit 1)
@@
 	)
 	(symbol
-		(lib_id "Device:C_Small")
+		(lib_id "minirex_g4:C_Small")
 		(at 46.99 26.67 0)
 		(unit 1)
@@
 	)
 	(symbol
-		(lib_id "power:+5V")
+		(lib_id "minirex_g4:+5V")
 		(at 170.18 35.56 270)
 		(unit 1)
@@
 	(symbol
 		(lib_name "R_Small_7")
-		(lib_id "Device:R_Small")
+		(lib_id "minirex_g4:R_Small_7")
 		(at 233.68 80.01 90)
 		(unit 1)
@@
 	)
 	(symbol
-		(lib_id "samacsys:LMR51625YFDDCR")
+		(lib_id "minirex_g4:LMR51625YFDDCR")
 		(at 85.09 40.64 0)
 		(unit 1)
@@
 	)
 	(symbol
-		(lib_id "power:GND")
+		(lib_id "minirex_g4:GND")
 		(at 209.55 81.28 90)
 		(unit 1)
@@
 	)
 	(symbol
-		(lib_id "samacsys2:74479335329247")
+		(lib_id "minirex_g4:74479335329247")
 		(at 118.11 35.56 0)
 		(unit 1)
@@
 	)
 	(symbol
-		(lib_id "power:GND")
+		(lib_id "minirex_g4:GND")
 		(at 60.96 29.21 0)
 		(unit 1)
@@
 	)
 	(symbol
-		(lib_id "power:GND")
+		(lib_id "minirex_g4:GND")
 		(at 210.82 124.46 90)
 		(unit 1)
@@
 	)
 	(symbol
-		(lib_id "power:GND")
+		(lib_id "minirex_g4:GND")
 		(at 250.19 80.01 90)
 		(unit 1)
@@
 	)
 	(symbol
-		(lib_id "power:PWR_FLAG")
+		(lib_id "minirex_g4:PWR_FLAG")
 		(at 148.59 36.83 0)
 		(unit 1)
@@
 	)
 	(symbol
-		(lib_id "power:GND")
+		(lib_id "minirex_g4:GND")
 		(at 88.9 97.79 90)
 		(unit 1)
@@
 	)
 	(symbol
-		(lib_id "Connector:TestPoint")
+		(lib_id "minirex_g4:TestPoint")
 		(at 80.01 132.08 0)
 		(unit 1)
@@
 	)
 	(symbol
-		(lib_id "samacsys2:SP3222-02ETG")
+		(lib_id "minirex_g4:SP3222-02ETG")
 		(at 114.3 106.68 0)
 		(unit 1)
@@
 	)
 	(symbol
-		(lib_id "Device:R_Small")
+		(lib_id "minirex_g4:R_Small")
 		(at 226.06 116.84 90)
 		(unit 1)
@@
 	)
 	(symbol
-		(lib_id "power:PWR_FLAG")
+		(lib_id "minirex_g4:PWR_FLAG")
 		(at 167.64 35.56 180)
 		(unit 1)
@@
 	)
 	(symbol
-		(lib_id "Vraielogousbcwurth:USB_C_Receptacle_USB2.0_14P")
+		(lib_id "minirex_g4:USB_C_Receptacle_USB2.0_14P")
 		(at 66.04 106.68 0)
 		(unit 1)
@@
 	)
 	(symbol
-		(lib_id "Device:C_Small")
+		(lib_id "minirex_g4:C_Small")
 		(at 144.78 39.37 0)
 		(unit 1)
@@
 	(symbol
 		(lib_name "R_Small_5")
-		(lib_id "Device:R_Small")
+		(lib_id "minirex_g4:R_Small_5")
 		(at 137.16 43.18 0)
 		(unit 1)
@@
 	)
 	(symbol
-		(lib_id "Connector:TestPoint")
+		(lib_id "minirex_g4:TestPoint")
 		(at 101.6 115.57 180)
 		(unit 1)
@@
 	)
 	(symbol
-		(lib_id "Device:C_Small")
+		(lib_id "minirex_g4:C_Small")
 		(at 250.19 133.35 0)
 		(unit 1)
@@
 	(symbol
 		(lib_name "R_Small_4")
-		(lib_id "Device:R_Small")
+		(lib_id "minirex_g4:R_Small_4")
 		(at 95.25 109.22 90)
 		(unit 1)
@@
 	)
 	(symbol
-		(lib_id "Device:C_Small")
+		(lib_id "minirex_g4:C_Small")
 		(at 66.04 26.67 0)
 		(unit 1)
@@
 	)
 	(symbol
-		(lib_id "power:GND")
+		(lib_id "minirex_g4:GND")
 		(at 193.04 142.24 0)
 		(unit 1)
@@
 	)
 	(symbol
-		(lib_id "Device:LED_Small")
+		(lib_id "minirex_g4:LED_Small")
 		(at 246.38 80.01 180)
 		(unit 1)
@@
 	)
 	(symbol
-		(lib_id "Connector:TestPoint")
+		(lib_id "minirex_g4:TestPoint")
 		(at 101.6 100.33 0)
 		(unit 1)
@@
 	)
 	(symbol
-		(lib_id "samacsys2:74279220800")
+		(lib_id "minirex_g4:74279220800")
 		(at 167.64 27.94 0)
 		(unit 1)
@@
 	)
 	(symbol
-		(lib_id "power:GND")
+		(lib_id "minirex_g4:GND")
 		(at 128.27 58.42 0)
 		(unit 1)
@@
 	(symbol
 		(lib_name "R_Small_2")
-		(lib_id "Device:R_Small")
+		(lib_id "minirex_g4:R_Small_2")
 		(at 83.82 99.06 90)
 		(unit 1)
@@
 	)
 	(symbol
-		(lib_id "power:PWR_FLAG")
+		(lib_id "minirex_g4:PWR_FLAG")
 		(at 219.71 85.09 180)
 		(unit 1)
@@
 	)
 	(symbol
-		(lib_id "samacsys:BAT60JFILM")
+		(lib_id "minirex_g4:BAT60JFILM")
 		(at 248.92 29.21 180)
 		(unit 1)
@@
 	(symbol
 		(lib_name "R_Small_1")
-		(lib_id "Device:R_Small")
+		(lib_id "minirex_g4:R_Small_1")
 		(at 83.82 96.52 90)
 		(unit 1)
@@
 	)
 	(symbol
-		(lib_id "power:GND")
+		(lib_id "minirex_g4:GND")
 		(at 166.37 96.52 0)
 		(unit 1)
@@
 	)
 	(symbol
-		(lib_id "Device:C_Small")
+		(lib_id "minirex_g4:C_Small")
 		(at 248.92 91.44 180)
 		(unit 1)
@@
 	(symbol
 		(lib_name "R_Small_3")
-		(lib_id "Device:R_Small")
+		(lib_id "minirex_g4:R_Small_3")
 		(at 95.25 106.68 90)
 		(unit 1)
@@
 	)
 	(symbol
-		(lib_id "samacsys2:LDL212PV33R")
+		(lib_id "minirex_g4:LDL212PV33R")
 		(at 209.55 81.28 0)
 		(mirror y)
@@
 	)
 	(symbol
-		(lib_id "Device:LED_Small")
+		(lib_id "minirex_g4:LED_Small")
 		(at 238.76 116.84 180)
 		(unit 1)
@@
 	)
 	(symbol
-		(lib_id "power:PWR_FLAG")
+		(lib_id "minirex_g4:PWR_FLAG")
 		(at 83.82 83.82 0)
 		(unit 1)
@@
 	)
 	(symbol
-		(lib_id "power:+5V")
+		(lib_id "minirex_g4:+5V")
 		(at 222.25 29.21 90)
 		(unit 1)
@@
 	)
 	(symbol
-		(lib_id "power:PWR_FLAG")
+		(lib_id "minirex_g4:PWR_FLAG")
 		(at 116.84 58.42 180)
 		(unit 1)
@@
 	)
 	(symbol
-		(lib_id "power:GND")
+		(lib_id "minirex_g4:GND")
 		(at 139.7 106.68 0)
 		(unit 1)
@@
 	)
 	(symbol
-		(lib_id "Device:C_Small")
+		(lib_id "minirex_g4:C_Small")
 		(at 115.57 25.4 0)
 		(unit 1)
@@
 	)
 	(symbol
-		(lib_id "power:GND")
+		(lib_id "minirex_g4:GND")
 		(at 191.77 99.06 0)
 		(unit 1)

Commit message: up
Parts:
- C12: Manufacturer_Name (none) -> Wurth Elektronik; Manufacturer_Part_Number (none) -> 885012104005; Mouser Part Number (none) -> 710-885012104005
- C13, C4: Manufacturer_Name (none) -> Murata; Manufacturer_Part_Number (none) -> GRT21BD72A225KE13; Mouser Part Number (none) -> 81-GRT21BD72A225KE13
- C17, C8: value 22u -> 47u; Manufacturer_Name (none) -> Murata; Manufacturer_Part_Number (none) -> GRM21BR61A476ME5K; Mouser Part Number (none) -> 81-GRM21BR61A476ME5K
- C2, C23: Manufacturer_Part_Number 885012105012 -> 885012105012; Mouser Part Number 710-885012105012 -> 710-885012105012
- C5: Manufacturer_Name (none) -> Murata; Manufacturer_Part_Number (none) -> GRM155R62A104ME4J; Mouser Part Number (none) -> 81-GRM155R62A104ME4J
- FB1: Manufacturer_Part_Number 74279220800 -> 710-74279220800
- J1: Manufacturer_Name GCT -> Wurth Elektronik; Manufacturer_Part_Number USB4110-GF-A -> 629722000214; Mouser Part Number 640-USB4110-GF-A -> 710-629722000214
- L1: Mouser Part Number (none) -> 710-74479335329247
- R11: Manufacturer_Name (none) -> Panasonic; Manufacturer_Part_Number (none) -> ERJ-1GNF1912C; Mouser Part Number (none) -> 667-ERJ-1GNF1912C
- R2: Manufacturer_Name (none) -> Panasonic; Manufacturer_Part_Number (none) -> ERJ-1GNF1003C; Mouser Part Number (none) -> 667-ERJ-1GNF1003C
Other:
- note added: "710-629722000214"
- note removed: "640-USB4110-GF-A"
- note removed: "GRM155R70J104KA01"
- note removed: "GRM21BZ71A226ME15"
- note removed: "GRM21BZ71E475ME15"
- note removed: "SP3222-02ETG"
