File: HARDWARE/V1/MINIREX_G4/MINIREX_G4.kicad_pcb (KiCad board)
At the start: 6 copper layers, 29 x 33 mm, 109 parts, among them IC1 ICM-42688-P, IC2 LMR51625YFDDCR, IC3 MX25R1635FZUIH0, IC4 LDL212PV33R, IC5 LDL212PV33R, J1 USB4110-GF-A, J2 SM08B-SRSS-TB, J3 SM06B-SRSS-TB, M1 TestPoint_Small, M2 TestPoint_Small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

Commit message: up
Parts:
- G***: footprint LOGO -> minirex_g4:LOGO
Other:
- board text removed: "1"
- board text removed: "2"
- board text removed: "3"
- board text removed: "4"
- board text removed: "DJI"
- board text removed: "ESC"
