File: HARDWARE/V1/MINIREX_G4/MINIREX_G4.kicad_sch (KiCad schematic)
At the start: 26 parts, among them Q1 2N7002KQBZ, U2 STM32G473CEUx, Y2 CSTNE8M00GH5C000R0

Commit message: up
Parts:
- C10, C11, C14, C16, C18, C19, C24, C26, C27, C6, C7, C9: symbol Device:C_Small -> minirex_g4:C_Small
- LEDBLUE1: symbol Device:LED_Small -> minirex_g4:LED_Small
- LEDGREEN1: symbol Device:LED_Small -> minirex_g4:LED_Small_1
- Q1: symbol samacsys:2N7002KQBZ -> minirex_g4:2N7002KQBZ
- R14: symbol Device:R_Small -> minirex_g4:R_Small_7
- R17: symbol Device:R_Small -> minirex_g4:R_Small_3
- R3: symbol Device:R_Small -> minirex_g4:R_Small
- R41: symbol Device:R_Small -> minirex_g4:R_Small_4
- R5: symbol Device:R_Small -> minirex_g4:R_Small_1
- R6: symbol Device:R_Small -> minirex_g4:R_Small_2
- R7: symbol Device:R_Small -> minirex_g4:R_Small_5
- R8: symbol Device:R_Small -> minirex_g4:R_Small_6
- S3: symbol samacsys:435151014824 -> minirex_g4:435151014824
- U2: symbol MCU_ST_STM32G4:STM32G473CEUx -> minirex_g4:STM32G473CEUx
- Y2: symbol samacsys:CSTNE8M00GH5C000R0 -> minirex_g4:CSTNE8M00GH5C000R0
Changed lines of the file:
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@@
 	)
 	(symbol
-		(lib_id "Device:C_Small")
+		(lib_id "minirex_g4:C_Small")
 		(at 172.72 53.34 0)
 		(unit 1)
@@
 	(symbol
 		(lib_name "R_Small_2")
-		(lib_id "Device:R_Small")
+		(lib_id "minirex_g4:R_Small_2")
 		(at 45.72 86.36 270)
 		(unit 1)
@@
 	)
 	(symbol
-		(lib_id "power:GND")
+		(lib_id "minirex_g4:GND")
 		(at 30.48 86.36 270)
 		(unit 1)
@@
 	)
 	(symbol
-		(lib_id "power:GND")
+		(lib_id "minirex_g4:GND")
 		(at 177.8 55.88 0)
 		(unit 1)
@@
 	)
 	(symbol
-		(lib_id "MCU_ST_STM32G4:STM32G473CEUx")
+		(lib_id "minirex_g4:STM32G473CEUx")
 		(at 201.93 124.46 0)
 		(unit 1)
@@
 	)
 	(symbol
-		(lib_id "Device:R_Small")
+		(lib_id "minirex_g4:R_Small")
 		(at 123.19 80.01 0)
 		(unit 1)
@@
 	)
 	(symbol
-		(lib_id "power:GND")
+		(lib_id "minirex_g4:GND")
 		(at 127 82.55 0)
 		(unit 1)
@@
 	)
 	(symbol
-		(lib_id "power:GND")
+		(lib_id "minirex_g4:GND")
 		(at 134.62 59.69 90)
 		(unit 1)
@@
 	)
 	(symbol
-		(lib_id "Device:C_Small")
+		(lib_id "minirex_g4:C_Small")
 		(at 180.34 63.5 0)
 		(unit 1)
@@
 	)
 	(symbol
-		(lib_id "Device:C_Small")
+		(lib_id "minirex_g4:C_Small")
 		(at 228.6 62.23 0)
 		(unit 1)
@@
 	)
 	(symbol
-		(lib_id "power:GND")
+		(lib_id "minirex_g4:GND")
 		(at 29.21 165.1 0)
 		(unit 1)
@@
 	)
 	(symbol
-		(lib_id "power:GND")
+		(lib_id "minirex_g4:GND")
 		(at 104.14 59.69 270)
 		(unit 1)
@@
 	)
 	(symbol
-		(lib_id "Device:C_Small")
+		(lib_id "minirex_g4:C_Small")
 		(at 189.23 53.34 0)
 		(unit 1)
@@
 	(symbol
 		(lib_name "R_Small_5")
-		(lib_id "Device:R_Small")
+		(lib_id "minirex_g4:R_Small_5")
 		(at 29.21 153.67 0)
 		(unit 1)
@@
 	)
 	(symbol
-		(lib_id "power:GND")
+		(lib_id "minirex_g4:GND")
 		(at 201.93 170.18 0)
 		(unit 1)
@@
 	)
 	(symbol
-		(lib_id "power:GND")
+		(lib_id "minirex_g4:GND")
 		(at 160.02 93.98 0)
 		(unit 1)
@@
 	(symbol
 		(lib_name "R_Small_7")
-		(lib_id "Device:R_Small")
+		(lib_id "minirex_g4:R_Small_7")
 		(at 60.96 153.67 0)
 		(unit 1)
@@
 	)
 	(symbol
-		(lib_id "Device:C_Small")
+		(lib_id "minirex_g4:C_Small")
 		(at 60.96 161.29 0)
 		(unit 1)
@@
 	)
 	(symbol
-		(lib_id "power:GND")
+		(lib_id "minirex_g4:GND")
 		(at 55.88 119.38 0)
 		(unit 1)
@@
 	)
 	(symbol
-		(lib_id "Device:C_Small")
+		(lib_id "minirex_g4:C_Small")
 		(at 162.56 53.34 0)
 		(unit 1)
@@
 	)
 	(symbol
-		(lib_id "Device:C_Small")
+		(lib_id "minirex_g4:C_Small")
 		(at 36.83 161.29 0)
 		(unit 1)
@@
 	)
 	(symbol
-		(lib_id "Device:C_Small")
+		(lib_id "minirex_g4:C_Small")
 		(at 181.61 53.34 0)
 		(unit 1)
@@
 	)
 	(symbol
-		(lib_id "power:GND")
+		(lib_id "minirex_g4:GND")
 		(at 161.29 76.2 0)
 		(unit 1)
@@
 	)
 	(symbol
-		(lib_id "Device:C_Small")
+		(lib_id "minirex_g4:C_Small")
 		(at 160.02 91.44 180)
 		(unit 1)
@@
 	)
 	(symbol
-		(lib_id "samacsys:CSTNE8M00GH5C000R0")
+		(lib_id "minirex_g4:CSTNE8M00GH5C000R0")
 		(at 54.61 48.26 270)
 		(mirror x)
@@
 	)
 	(symbol
-		(lib_id "samacsys:435151014824")
+		(lib_id "minirex_g4:435151014824")
 		(at 104.14 59.69 0)
 		(unit 1)
@@
 	(symbol
 		(lib_name "R_Small_3")
-		(lib_id "Device:R_Small")
+		(lib_id "minirex_g4:R_Small_3")
 		(at 43.18 105.41 90)
 		(unit 1)
@@
 	)
 	(symbol
-		(lib_id "power:GND")
+		(lib_id "minirex_g4:GND")
 		(at 180.34 66.04 0)
 		(unit 1)
@@
 	)
 	(symbol
-		(lib_id "power:GND")
+		(lib_id "minirex_g4:GND")
 		(at 60.96 165.1 0)
 		(unit 1)
@@
 	)
 	(symbol
-		(lib_id "Device:C_Small")
+		(lib_id "minirex_g4:C_Small")
 		(at 237.49 62.23 0)
 		(unit 1)
@@
 	(symbol
 		(lib_name "R_Small_1")
-		(lib_id "Device:R_Small")
+		(lib_id "minirex_g4:R_Small_1")
 		(at 45.72 80.01 270)
 		(unit 1)
@@
 	)
 	(symbol
-		(lib_id "Device:C_Small")
+		(lib_id "minirex_g4:C_Small")
 		(at 130.81 80.01 180)
 		(unit 1)
@@
 	(symbol
 		(lib_name "LED_Small_1")
-		(lib_id "Device:LED_Small")
+		(lib_id "minirex_g4:LED_Small_1")
 		(at 33.02 80.01 0)
 		(unit 1)
@@
 	(symbol
 		(lib_name "R_Small_6")
-		(lib_id "Device:R_Small")
+		(lib_id "minirex_g4:R_Small_6")
 		(at 29.21 161.29 0)
 		(unit 1)
@@
 	)
 	(symbol
-		(lib_id "power:GND")
+		(lib_id "minirex_g4:GND")
 		(at 52.07 48.26 0)
 		(unit 1)
@@
 	)
 	(symbol
-		(lib_id "power:PWR_FLAG")
+		(lib_id "minirex_g4:PWR_FLAG")
 		(at 218.44 59.69 0)
 		(unit 1)
@@
 	)
 	(symbol
-		(lib_id "Device:C_Small")
+		(lib_id "minirex_g4:C_Small")
 		(at 161.29 73.66 180)
 		(unit 1)
@@
 	)
 	(symbol
-		(lib_id "power:GND")
+		(lib_id "minirex_g4:GND")
 		(at 30.48 80.01 270)
 		(unit 1)
@@
 	(symbol
 		(lib_name "R_Small_4")
-		(lib_id "Device:R_Small")
+		(lib_id "minirex_g4:R_Small_4")
 		(at 45.72 111.76 0)
 		(unit 1)
@@
 	)
 	(symbol
-		(lib_id "samacsys:2N7002KQBZ")
+		(lib_id "minirex_g4:2N7002KQBZ")
 		(at 55.88 105.41 0)
 		(unit 1)
@@
 	)
 	(symbol
-		(lib_id "power:GND")
+		(lib_id "minirex_g4:GND")
 		(at 233.68 64.77 0)
 		(unit 1)
@@
 	)
 	(symbol
-		(lib_id "Device:LED_Small")
+		(lib_id "minirex_g4:LED_Small")
 		(at 33.02 86.36 0)
 		(unit 1)
@@
 		)
 		(instances
-			(project "FC_H7_MINI"
+			(project "MINIREX_G4"
 				(path "/61daacfc-87c7-44e7-aaaa-5f4739cb2045"
 					(page "2")
@@
 		)
 		(instances
-			(project "FC_H7_MINI"
+			(project "MINIREX_G4"
 				(path "/61daacfc-87c7-44e7-aaaa-5f4739cb2045"
 					(page "3")
@@
 		)
 		(instances
-			(project "FC_H7_MINI"
+			(project "MINIREX_G4"
 				(path "/61daacfc-87c7-44e7-aaaa-5f4739cb2045"
 					(page "4")

Commit message: up
Parts:
- C6: Manufacturer_Part_Number 885012105008 -> 885012105012; Mouser Part Number 710-885012105008 -> 710-885012105012
- U2: Manufacturer_Name (none) -> STMicroelectronics; Manufacturer_Part_Number (none) -> STM32G473CEU6; Mouser Part Number (none) -> 511-STM32G473CEU6

Commit message: picture add
Changed lines of the file:
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@@
 	)
 	(sheet
-		(at 307.34 58.42)
+		(at 269.24 54.61)
 		(size 45.72 25.4)
 		(exclude_from_sim no)
@@
 		)
 		(property "Sheetname" "Peripherials onboard"
-			(at 307.34 57.7084 0)
+			(at 269.24 53.8984 0)
 			(effects
 				(font
@@
 		)
 		(property "Sheetfile" "Peripherials.kicad_sch"
-			(at 307.34 84.4046 0)
+			(at 269.24 80.5946 0)
 			(effects
 				(font
@@
 	)
 	(sheet
-		(at 307.34 95.25)
+		(at 269.24 91.44)
 		(size 44.45 26.67)
 		(exclude_from_sim no)
@@
 		)
 		(property "Sheetname" "Power supply"
-			(at 307.34 94.5384 0)
+			(at 269.24 90.7284 0)
 			(effects
 				(font
@@
 		)
 		(property "Sheetfile" "untitled.kicad_sch"
-			(at 307.34 122.5046 0)
+			(at 269.24 118.6946 0)
 			(effects
 				(font
@@
 	)
 	(sheet
-		(at 307.34 135.89)
+		(at 269.24 132.08)
 		(size 44.45 24.13)
 		(exclude_from_sim no)
@@
 		)
 		(property "Sheetname" "Connectors"
-			(at 307.34 135.1784 0)
+			(at 269.24 131.3684 0)
 			(effects
 				(font
@@
 		)
 		(property "Sheetfile" "connectors.kicad_sch"
-			(at 307.34 160.6046 0)
+			(at 269.24 156.7946 0)
 			(effects
 				(font
