File: HARDWARE/V2/MINIREX_G4/MINIREX_G4.kicad_pcb (KiCad board)
At the start: 6 copper layers, 29 x 33 mm, 109 parts, among them IC1 ICM-42688-P, IC2 LMR51625YFDDCR, IC3 MX25R1635FZUIH0, IC4 LDL212PV33R, IC5 LDL212PV33R, J1 USB4110-GF-A, J2 SM08B-SRSS-TB, J3 SM06B-SRSS-TB, M1 TestPoint_Small, M2 TestPoint_Small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

Commit message: up
Parts:
- removed Q1: 2N7002KQBZ, samacsys:2N7002KQBZ
- removed S3: 435151014824, samacsys:435151014824
- added Q2: PMZB150UNEYL, samacsys2:PMZB150UNEYL, F.Cu at (91.4, 97.4)
- added S1: TS2306A-240GF-MSM-9_C388290, samacsys2:TS2306A240GFMSM9_C388290, F.Cu at (95.0, 101.5)
- C17, C8: value 22u -> 47u
- C22: value 10n -> 100n
- D1: value SP3222-02ETG -> TPSP3222-02ETG
- FB1: value 74279220800 -> MPZ2012S101ATD25
- IC1: value ICM-42688-P -> ICM-42688P
- IC3: value MX25R1635FZUIH0 -> ZD25WQ32CEIGR
- J1: value USB4110-GF-A -> USB4105-GF-A
- L1: value 74479335329247 -> ZEPIM303020D-4R7M
- R13, R44, R45, R46, R47, R56, R61: value 22R -> 47R
- R15, R3, R9: value 10k -> 19.1k
- R17: value 100R -> 47R
- R7: value 20k -> 19.1k
Routing:
- net GND: track 10.3 -> 6.46 mm
- net 3.3VMCU: track 7.91 -> 4.59 mm
- net Rx2: track 7.45 -> 8.04 mm
- net BUZ-: vias 2 -> 1
