File: HARDWARE/V2/MINIREX_G4/MINIREX_G4.kicad_pcb (KiCad board)
At the start: 6 copper layers, 29 x 33 mm, 109 parts, among them IC1 ICM-42688P, IC2 LMR51625YFDDCR, IC3 ZD25WQ32CEIGR, IC4 LDL212PV33R, IC5 LDL212PV33R, J1 USB4105-GF-A, J2 SM08B-SRSS-TB, J3 SM06B-SRSS-TB, M1 TestPoint_Small, M2 TestPoint_Small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

Commit message: up
Parts:
- moved C5 5.77 mm to (85.8, 86.1), turned to 180 degrees
- moved C21 0.94 mm to (103.9, 88.7)
- moved R7 0.90 mm to (87.7, 86.2)
- moved C14 0.83 mm to (88.2, 87.8)
- moved R9 0.78 mm to (88.1, 88.6)
- moved R1 0.43 mm to (83.7, 86.3)
- moved C10 0.40 mm to (90.3, 87.0)
- moved C13 0.29 mm to (85.0, 84.7)
- moved C4 0.28 mm to (85.0, 82.7)
- moved IC3 0.14 mm to (85.1, 88.0)
- moved C7 0.09 mm to (95.6, 97.3)
- moved C3 0.06 mm to (102.4, 87.4)
Routing:
- net 3.3VMCU: track 4.59 -> 15.6 mm
- net GND: track 6.69 -> 9.83 mm, vias 189 -> 183
- net ADC_VBAT: track 8.17 -> 9.16 mm
- net FLASH_CS/SPI2: track 4.07 -> 3.26 mm
- net Net-(J2-Pad3): track 33.1 -> 33.9 mm
- net Net-(J2-Pad4): track 33.6 -> 34.2 mm
- net Net-(J2-Pad6): track 38.4 -> 39.0 mm
- net Net-(J2-Pad5): track 35.9 -> 36.4 mm
Other:
- board text added: "vusb"
